Commit message: 키보드 조작 반절 성공

File: my_robot.urdf (robot description, URDF)
Before this commit: robot my_robot, 7 links, 6 joints
Links:
- link link1: mass None -> 0.090
- link link2: mass None -> 0.090
- link link3: mass None -> 0.090
- link link4: mass None -> 0.090
- link link5: mass None -> 0.050
Joints:
- joint joint1: limit lower=0 upper=3.14159 effort=1.0 velocity=1.0 -> lower=0.1745 upper=2.9671 effort=1.47 velocity=1.0; origin xyz=0 0 0.05 rpy=0 0 0 -> xyz=0 0 0.088 rpy=0 0 0
- joint joint2: limit lower=0 upper=3.14159 effort=1.0 velocity=1.0 -> lower=0.1745 upper=2.9671 effort=2.1 velocity=1.0; origin xyz=0 0 0 rpy=0 0 0 -> xyz=-0.022 0 0 rpy=0 -1.5707 0
- joint joint3: axis 0 1 0 -> 0 -1 0; limit lower=0 upper=3.14159 effort=1.0 velocity=1.0 -> lower=0.1745 upper=2.9671 effort=1.47 velocity=1.0; origin xyz=0 0 0.104 rpy=0 0 0 -> xyz=0.104 0 0 rpy=0 0 0
- joint joint4: limit lower=0 upper=3.14159 effort=1.0 velocity=1.0 -> lower=0.1745 upper=2.9671 effort=1.47 velocity=1.0; origin xyz=0 0 0.125 rpy=0 0 0 -> xyz=0.125 0 0 rpy=0 0 0
- joint joint5: limit lower=0 upper=3.14159 effort=1.0 velocity=1.0 -> lower=0.1745 upper=2.9671 effort=1.47 velocity=1.0
- joint tcp_joint: origin xyz=0.182 0 0 rpy=0 0 0 -> xyz=0.162 0 0 rpy=0 0 0
